File: board.brd (EAGLE design)
At the start: 100 x 80 mm, 0 parts

Commit message: Schematics v1
Parts:
- added C1: 470u, rcl:E3,5-8
- added C2, C3, C5: 0.1u, rcl:C0805
- added C4: 100n, rcl:C0805
- added D1, D3, D4, D5, D6: STTH4R02UY, diode:SMB
- added F1, F2, F3: 1.6A, fuse:SHK20L
- added F4, F5, F9: 30V/1.6A, SparkFun-Fuses:PTH
- added F6, F7, F8: 30V/4A, SparkFun-Fuses:PTH
- added IC1: REG1117, burr-brown:SOT223
- added J1: LHBEAMOUT, SparkFun-Connectors:SCREWTERMINAL-3.5MM-3
- added J10: ATEMP, SparkFun-Connectors:SCREWTERMINAL-3.5MM-2
- added J11: HORNOUT, SparkFun-Connectors:SCREWTERMINAL-3.5MM-2
- added J12: 12V_SUPPLY, SparkFun-Connectors:SCREWTERMINAL-3.5MM-2
- added J13: STOPOUT, SparkFun-Connectors:SCREWTERMINAL-3.5MM-2
- added J14: TURNOUT, SparkFun-Connectors:SCREWTERMINAL-3.5MM-3
- added J15: FANOUT, SparkFun-Connectors:SCREWTERMINAL-3.5MM-2
- added J16: BLIGHTOUT, SparkFun-Connectors:SCREWTERMINAL-3.5MM-2
- added J17: AUXOUT, SparkFun-Connectors:SCREWTERMINAL-3.5MM-2
- added J18: AUX, SparkFun-Connectors:SCREWTERMINAL-3.5MM-2
- added J19: CAN, SparkFun-Connectors:SCREWTERMINAL-3.5MM-2
- added J2: BATT, SparkFun-Connectors:SCREWTERMINAL-3.5MM-2
- added J3: BLIGHT, SparkFun-Connectors:SCREWTERMINAL-3.5MM-2
- added J4: LHBEAM, SparkFun-Connectors:SCREWTERMINAL-3.5MM-3
- added J5: LRTURN, SparkFun-Connectors:SCREWTERMINAL-3.5MM-3
- added J6: WARNING, SparkFun-Connectors:SCREWTERMINAL-3.5MM-2
- added J7: HORN, SparkFun-Connectors:SCREWTERMINAL-3.5MM-2
- added J8: BREAK, SparkFun-Connectors:SCREWTERMINAL-3.5MM-2
- added J9: ABREAK, SparkFun-Connectors:SCREWTERMINAL-3.5MM-2
- added L1: 15uH, inductor-bourns:SDR1307
- added Q1, Q2, Q3: IRF7465TR, transistor-power:SO-08
- added Q4: IRLML9301TRPBF, svetozar:SC75_INFINEON
- added Q5, Q9: IRLML9301TRPBF, my:SC75_INFINEON
- added Q6, Q7, Q8: IRF7424TRPBF, transistor-power:SO-08
- added R1, R2, R3: 160, rcl:R0805
- added R10, R11, R12, R4, R5, R6, R7, R8, R9: 1k, rcl:R0805
- added R13: 3k, rcl:R0805
- added R14: 2.4k, rcl:R0805
- added R15: 10k, rcl:R0805
- added U$1: (no value), BluePill:BLUE_PILL
- added U1, U2, U3: VOM1271T, VOM1271T:SOIC254P695X242-4N
- added U4: MC14504BDR2G, MC14504BDR2G:SOIC127P600X175-16N
- added U5: MAX3051ESA, MAX3051ESA:8-SOICN
Connections:
- new net +12V: C2.1, F4.P$2, F5.P$2, F6.P$2, F7.P$2, F8.P$2, F9.P$2, IC1.3, J12.1, U4.16
- new net +3V3: C3.1, C5.1, IC1.2, R10.1, R11.1, R12.1, R14.1, R4.1, R5.1, R6.1, R7.1, R8.1, R9.1, U$1.P$20, U$1.P$23, U4.1, U5.3
- new net AUXOUT: D1.C, J17.1, Q8.5, Q8.6, Q8.7, Q8.8
- new net BATT+: F1.2A, F2.2A, F3.2A, J2.1
- new net BATT-: D4.A, D5.A, D6.A, J1.3, J11.2, J2.2
- new net BLIGHTOUT: J16.1, Q7.5, Q7.6, Q7.7, Q7.8
- new net CANH: J19.1, U5.7
- new net CANL: J19.2, U5.6
- new net FANOUT: C1.+, D3.C, J15.1, L1.2
- new net GND: C4.2, C5.2, J10.1, J18.1, J3.1, J4.1, J5.1, J6.1, J7.1, J8.1, J9.1, R15.2, U5.2, U5.8
- new net GND1: C1.-, C2.2, C3.2, D1.A, D3.A, IC1.1, J12.2, J13.2, J14.3, J15.2, J16.2, J17.2, U$1.P$19, U$1.P$21, U$1.P$22, U1.2, U2.2, U3.2, U4.13, U4.8
- new net HBEAMOUT: D5.C, J1.2, Q2.1, Q2.2, Q2.3, U2.3
- new net HORNOUT: D6.C, J11.1, Q3.1, Q3.2, Q3.3, U3.3
- new net HV1CTL: R1.1, U$1.P$27
- new net HV2CTL: R2.1, U$1.P$28
- new net HV3CTL: R3.1, U$1.P$29
- new net LBEAMOUT: D4.C, J1.1, Q1.1, Q1.2, Q1.3, U1.3
- new net LTURNOUT: J14.1, Q5.2
- new net LVCTL1: U$1.P$30, U4.3
- new net N$1: U$1.P$33, U4.5
- new net N$10: F1.1A, Q1.5, Q1.6, Q1.7, Q1.8
- new net N$11: F2.1A, Q2.5, Q2.6, Q2.7, Q2.8
- new net N$12: F3.1A, Q3.5, Q3.6, Q3.7, Q3.8
- new net N$13: U$1.P$15, U4.11
- new net N$14: U$1.P$14, U4.14
- new net N$15: J3.2, R4.2, U$1.P$36
- new net N$16: F4.P$1, Q4.3
- new net N$17: L1.1, Q6.5, Q6.6, Q6.7, Q6.8
- new net N$18: F5.P$1, Q5.3
- new net N$19: F6.P$1, Q6.1, Q6.2, Q6.3
- new net N$2: U$1.P$34, U4.7
- new net N$20: Q4.1, U4.2
- new net N$21: F7.P$1, Q7.1, Q7.2, Q7.3
- new net N$22: F8.P$1, Q8.1, Q8.2, Q8.3
- new net N$23: F9.P$1, Q9.3
- new net N$24: Q5.1, U4.4
- new net N$25: Q9.1, U4.6
- new net N$26: Q6.4, U4.10
- new net N$27: Q7.4, U4.12
- new net N$28: Q8.4, U4.15
- new net N$29: J4.3, R6.2, U$1.P$1
- new net N$3: U$1.P$35, U4.9
- new net N$30: J4.2, R5.2, U$1.P$2
- new net N$31: J7.2, R10.2, U$1.P$6
- new net N$32: J5.3, R8.2, U$1.P$3
- new net N$33: J5.2, R7.2, U$1.P$4
- new net N$34: J8.2, R11.2, U$1.P$7
- new net N$35: J6.2, R9.2, U$1.P$5
- new net N$36: J18.2, R12.2, U$1.P$10
- new net N$37: C4.1, J10.2, R14.2, U$1.P$32
- new net N$38: J9.2, R13.1
- new net N$39: R13.2, R15.1, U$1.P$31
- new net N$4: R1.2, U1.1
- new net N$40: U$1.P$16, U5.4
- new net N$41: U$1.P$17, U5.1
- new net N$42: U$1.P$13, U5.5
- new net N$5: R2.2, U2.1
- new net N$6: R3.2, U3.1
- new net N$7: Q1.4, U1.4
- new net N$8: Q2.4, U2.4
- new net N$9: Q3.4, U3.4
- new net RTURNOUT: J14.2, Q9.2
- new net STOPOUT: J13.1, Q4.2

Commit message: PCB v.1
Parts:
- added C6: 470u, rcl:E3,5-8
- added C7: 47u6V, rcl:C1206
- added C8: 22u16V, rcl:C1206
- added LOGO2: OSHW-LOGOL, SparkFun-Aesthetics:OSHW-LOGO-L
- added R16: 120, rcl:R0805
- C4: value 100n -> 0.1u
- F6, F7, F8: value 30V/4A -> 30V4A; device SparkFun-Fuses:PTH -> svetozar:PTH
- IC1: value REG1117 -> LM1117; device burr-brown:SOT223 -> svetozar:SOT223
- U5: value MAX3051ESA -> MAX3051ESA+T; device MAX3051ESA:8-SOICN -> MAX3051ESA:SO-08
- moved J19 760.3 mm to (11.2, 78.5), turned to 270 degrees
- moved C5 757.0 mm to (31.5, 78.3), turned to 270 degrees
- moved U5 745.4 mm to (26.5, 77.6), turned to 90 degrees
- moved R15 741.0 mm to (15.7, 73.4), turned to 90 degrees
- moved C4 726.4 mm to (15.7, 64.7), turned to 90 degrees
- moved R13 719.6 mm to (15.7, 69.3), turned to 90 degrees
- moved R14 716.2 mm to (15.7, 60.7), turned to 90 degrees
- moved R6 666.4 mm to (15.7, 50.4), turned to 90 degrees
- moved R8 666.4 mm to (15.7, 40.2), turned to 90 degrees
- moved R5 666.4 mm to (15.7, 55.4), turned to 90 degrees
- moved R7 666.4 mm to (15.7, 45.3), turned to 90 degrees
- moved R9 665.8 mm to (15.7, 34.5), turned to 90 degrees
- moved R10 663.9 mm to (15.7, 27.5), turned to 90 degrees
- moved R11 662.0 mm to (15.7, 20.5), turned to 90 degrees
- moved R12 660.2 mm to (15.7, 13.5), turned to 90 degrees
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Connections:
- net N$10 renamed HV1
- net N$11 renamed HV2
- net N$12 renamed HV3
- net N$40 renamed CANRX
- net N$41 renamed CANTX
- net N$42 renamed CANSHDN
- removed net GND1: C1.-, C2.2, C3.2, D1.A, D3.A, IC1.1, J12.2, J13.2, J14.3, J15.2, J16.2, J17.2, U$1.P$19, U$1.P$21, U$1.P$22, U1.2, U2.2, U3.2, U4.13, U4.8
- net +12V: now also C6.+, C8.1
- net +3V3: now also C7.1, IC1.4
- net CANH: now also J19.2, R16.2; no longer J19.1
- net CANL: now also J19.1, R16.1; no longer J19.2
- net GND: now also C1.-, C2.2, C3.2, C6.-, C7.2, C8.2, D1.A, D3.A, IC1.1, J12.2, J13.2, J14.3, J15.2, J16.2, J17.2, U$1.P$19, U$1.P$21, U$1.P$22, U1.2, U2.2, U3.2, U4.13, U4.8
- net N$1: now also U4.9; no longer U4.5
- net N$13: now also U4.5; no longer U4.11
- net N$14: now also U4.7; no longer U4.14
- net N$2: now also U4.11; no longer U4.7
- net N$24: now also Q9.1; no longer Q5.1
- net N$25: now also Q5.1; no longer Q9.1
- net N$26: now also U4.12; no longer U4.10
- net N$27: now also U4.10; no longer U4.12
- net N$29: now also U$1.P$2; no longer U$1.P$1
- net N$3: now also U4.14; no longer U4.9
- net N$30: now also U$1.P$1; no longer U$1.P$2
- net N$32: now also U$1.P$4; no longer U$1.P$3
- net N$33: now also U$1.P$3; no longer U$1.P$4
Routing:
- net GND: track 0.00 -> 379.2 mm, vias 0 -> 2
- net +3V3: track 0.00 -> 147.1 mm, vias 0 -> 1
- net +12V: track 0.00 -> 122.5 mm
- net BATT+: track 0.00 -> 58.9 mm
- net N$15: track 0.00 -> 58.3 mm
- net N$34: track 0.00 -> 55.2 mm
- net N$36: track 0.00 -> 54.0 mm
- net BATT-: track 0.00 -> 52.4 mm
- net N$31: track 0.00 -> 51.0 mm
- net N$20: track 0.00 -> 48.8 mm, vias 0 -> 2
- net N$35: track 0.00 -> 46.6 mm
- net N$25: track 0.00 -> 45.9 mm, vias 0 -> 2
- net N$24: track 0.00 -> 45.5 mm, vias 0 -> 2
- net CANRX: track 0.00 -> 43.2 mm, vias 0 -> 1
- net N$33: track 0.00 -> 42.4 mm
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Other:
- board size 100 x 80 mm -> 76 x 83.5 mm
- board text added: "12-130V"
- board text added: "12V"
- board text added: "ABRK"
- board text added: "ATEMP"
- board text added: "AUX"
- board text added: "BATT+"
- board text added: "BATT-"
- board text added: "BATT–"
- board text added: "BLGHT"
- board text added: "BRK"
- board text added: "CANH"
- board text added: "CANL"
- board text added: "FAN"
- board text added: "GND"
- board text added: "HBEAM"
- board text added: "HORN"
- board text added: "INPUTS"
- board text added: "LBEAM"
- board text added: "LEFT"
- board text added: "LTURN"
- board text added: "OUTPUTS"
- board text added: "RGHT"
- board text added: "RTURN"
- board text added: "STOP"
- board text added: "WARN"
- board text added: "https://github.com/ryba-xek/Svetozar"
- board text added: "v.1"

Commit message: Board & schematics v 1.1. Minor improvements
Parts:
- C2: device rcl:C0805 -> rcl:C1206
- moved C2 5.79 mm to (34.8, 27.7), turned to 270 degrees
- moved C3 4.44 mm to (19.7, 29.2), turned to 0 degrees
- moved R2 3.18 mm to (30.9, 64.9)
- moved Q9 2.32 mm to (60.1, 8.55)
- moved R1 2.16 mm to (30.9, 62.1)
- moved Q5 1.82 mm to (60.1, 4.86)
- moved Q4 1.69 mm to (60.1, 11.3)
- moved C6 1.42 mm to (23.5, 14.6)
- moved D3 1.17 mm to (48.3, 19.6)
- moved LOGO2 0.85 mm to (21.8, 5.59)
- moved Q6 0.28 mm to (38.8, 21.4)
- moved C7 0.28 mm to (30.9, 13.8)
- moved C8 0.25 mm to (30.9, 16.0)
- moved IC1 0.25 mm to (30.1, 7.15)
Connections:
- net N$1 renamed LVCTL4
- net N$13 renamed LVCTL2
- net N$14 renamed LVCTL3
- net N$2 renamed LVCTL5
- net N$20 renamed LV4G
- net N$24 renamed LV5G
- net N$25 renamed LV6G
- net N$26 renamed LV3G
- net N$27 renamed LV2G
- net N$28 renamed LV1G
- net N$3 renamed LVCTL6
- net N$37 renamed IATEMP
- net N$38 renamed ABRK
- net N$39 renamed ABRK_S
- net N$4 renamed HV1CTLG
- net N$5 renamed HV2CTLG
- net N$6 renamed HV3CTLG
- net N$7 renamed HV1G
- net N$8 renamed HV2G
- net N$9 renamed HV3G
- net HV1CTL: now also U$1.P$28; no longer U$1.P$27
- net HV2CTL: now also U$1.P$27; no longer U$1.P$28
Routing:
- net GND: track 379.2 -> 356.4 mm
- net +12V: track 122.5 -> 112.2 mm
- net HV2CTLG: track 21.9 -> 13.6 mm
- net N$17: track 13.4 -> 19.0 mm
- net LVCTL2: track 27.7 -> 23.1 mm, vias 2 -> 0
- net BATT-: track 52.4 -> 49.2 mm
- net HV1CTLG: track 13.9 -> 11.0 mm
- net +3V3: track 147.1 -> 144.6 mm, vias 1 -> 2
- net BATT+: track 58.9 -> 56.5 mm
- net LV4G: track 48.8 -> 46.9 mm
- net STOPOUT: track 7.68 -> 5.91 mm
- net LVCTL1: track 38.8 -> 37.3 mm
- net N$19: track 6.38 -> 7.79 mm
- net RTURNOUT: track 5.58 -> 4.18 mm
- net N$15: track 58.3 -> 56.9 mm
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Other:
- board text added: "6.10.2018"
- board text added: "v.1.1"
- board text removed: "v.1"

Commit message: WIP
Parts:
- removed F1, F2, F3: 1.6A, fuse:SHK20L
- removed F4, F5, F9: 30V/1.6A, SparkFun-Fuses:PTH
- removed F6, F7, F8: 30V4A, svetozar:PTH
- added C10, C9: 1n, rcl:C0805
- added C11, C12: 0.1u, rcl:C0805
- added JP1: (no value), jumper:JP1
- added JP2: (no value), jumper:JP2
- added LED1: (no value), led:SML0805
- added R17: 1k, rcl:R0603
- added R18, R19, R20, R21, R22, R23: 10k, rcl:R0603
- added U$2, U$3: ACS711LC, svetozar:SO08
- C1, C6: device rcl:E3,5-8 -> rcl:PANASONIC_F
- IC1: value LM1117 -> REG1117F; device svetozar:SOT223 -> burr-brown:DD-3
- J10: value ATEMP -> TEMP
- J8: value BREAK -> (none); device SparkFun-Connectors:SCREWTERMINAL-3.5MM-2 -> SparkFun-Connectors:1X01
- J9: value ABREAK -> BREAK; device SparkFun-Connectors:SCREWTERMINAL-3.5MM-2 -> SparkFun-Connectors:SCREWTERMINAL-3.5MM-3
- Q1, Q2, Q3: value IRF7465TR -> FQD19N10LTM; device transistor-power:SO-08 -> SparkFun-DiscreteSemi:DPAK
- Q4: value IRLML9301TRPBF -> IRF7424TRPBF; device svetozar:SC75_INFINEON -> transistor-power:SO-08
- Q5, Q9: value IRLML9301TRPBF -> IRF7424TRPBF; device my:SC75_INFINEON -> transistor-power:SO-08
- R10, R12, R13, R14, R15, R4, R5, R6, R7, R8, R9: device rcl:R0805 -> rcl:R0603
- moved IC1 71.4 mm to (46.1, 76.7), turned to 0 degrees
- moved C6 61.2 mm to (56.5, 66.2)
- moved R15 57.9 mm to (19.3, 15.6)
- moved J9 57.5 mm to (11.0, 14.0)
- moved C8 56.2 mm to (50.8, 68.6), turned to 270 degrees
- moved R13 54.5 mm to (16.5, 14.8), turned to 0 degrees
- moved J8 53.9 mm to (40.0, 67.9), turned to 0 degrees
- moved C7 53.7 mm to (49.5, 64.1)
- moved C4 46.2 mm to (15.7, 18.5), turned to 270 degrees
- moved R11 44.6 mm to (44.5, 54.6), turned to 180 degrees
- moved J10 43.5 mm to (11.0, 21.0)
- moved R14 38.3 mm to (15.7, 22.4), turned to 270 degrees
- moved R4 36.2 mm to (15.7, 42.9), turned to 270 degrees
- moved U3 36.0 mm to (41.9, 77.5), flipped to the bottom, turned to 270 degrees
- moved D6 33.7 mm to (41.9, 70.5), flipped to the bottom, turned to 0 degrees
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Connections:
- net ABRK renamed N$5
- removed net CANL: J19.1, R16.1, U5.6
- removed net HV1: F1.1A, Q1.5, Q1.6, Q1.7, Q1.8
- removed net HV2: F2.1A, Q2.5, Q2.6, Q2.7, Q2.8
- removed net HV3: F3.1A, Q3.5, Q3.6, Q3.7, Q3.8
- removed net N$15: J3.2, R4.2, U$1.P$36
- removed net N$16: F4.P$1, Q4.3
- removed net N$18: F5.P$1, Q5.3
- removed net N$19: F6.P$1, Q6.1, Q6.2, Q6.3
- removed net N$21: F7.P$1, Q7.1, Q7.2, Q7.3
- removed net N$22: F8.P$1, Q8.1, Q8.2, Q8.3
- removed net N$23: F9.P$1, Q9.3
- removed net N$34: J8.2, R11.2, U$1.P$7
- removed net N$36: J18.2, R12.2, U$1.P$10
- new net BATT+IN: J2.1, U$2.1, U$2.2
- new net CSENS1: C9.1, U$1.P$36, U$2.7
- new net FAULT: R11.1, U$1.P$11, U$2.6, U$3.6
- new net IAUX: J18.2, R12.2, U$1.P$12
- new net IBLGHT: J3.2, R4.2, U$1.P$25
- new net N$1: JP1.2, R16.1
- new net N$2: J19.1, JP1.1, U5.6
- new net N$3: JP2.1, R13.2, R15.1
- new net N$4: J9.3, JP2.3, R17.2
- new net N$6: J8.1, LED1.A, U$1.P$26
- new net N$7: J12.1, U$3.1, U$3.2
- new net N$8: C10.1, U$1.P$30, U$3.7
- new net N$9: C11.1, C12.1, U$1.P$10, U$2.8, U$3.8
- net +12V: now also Q4.1, Q4.2, Q4.3, Q5.1, Q5.2, Q5.3, Q6.1, Q6.2, Q6.3, Q7.1, Q7.2, Q7.3, Q8.1, Q8.2, Q8.3, Q9.1, Q9.2, Q9.3, U$3.3, U$3.4; no longer F4.P$2, F5.P$2, F6.P$2, F7.P$2, F8.P$2, F9.P$2, J12.1
- net +3V3: now also R11.2, R17.1, R18.2, R19.2, R20.2, R21.2, R22.2, R23.2; no longer IC1.4, R11.1
- net ABRK_S: now also JP2.2; no longer R13.2, R15.1
- net BATT+: now also Q1.4, Q2.4, Q3.4, U$2.3, U$2.4; no longer F1.2A, F2.2A, F3.2A, J2.1
- net FANOUT: no longer D3.C
- net GND: now also C10.2, C11.2, C12.2, C9.2, LED1.C, U$2.5, U$3.5; no longer J8.1
- net HBEAMOUT: no longer Q2.1, Q2.2
- net HORNOUT: no longer Q3.1, Q3.2
- net HV1G: now also Q1.1; no longer Q1.4
- net HV2G: now also Q2.1; no longer Q2.4
- net HV3G: now also Q3.1; no longer Q3.4
- net LBEAMOUT: no longer Q1.1, Q1.2
- net LTURNOUT: now also Q5.5, Q5.6, Q5.7, Q5.8; no longer Q5.2
- net LV4G: now also Q4.4; no longer Q4.1
- net LV5G: now also Q9.4; no longer Q9.1
- net LV6G: now also Q5.4; no longer Q5.1
- net LVCTL1: now also R23.1, U$1.P$7; no longer U$1.P$30
- net LVCTL2: now also R22.1
- net LVCTL3: now also R21.1
- net LVCTL4: now also R20.1
- net LVCTL5: now also R19.1
- net LVCTL6: now also R18.1
- net N$17: now also D3.C
- net RTURNOUT: now also Q9.5, Q9.6, Q9.7, Q9.8; no longer Q9.2
- net STOPOUT: now also Q4.5, Q4.6, Q4.7, Q4.8; no longer Q4.2
Routing:
- net GND: track 356.4 -> 22.6 mm
- net +12V: track 112.2 -> 2.54 mm
- net +3V3: track 144.6 -> 69.3 mm, vias 2 -> 14
- net N$15: track 56.9 -> 0.00 mm
- net N$34: track 55.2 -> 0.00 mm
- net N$36: track 54.0 -> 0.00 mm
- net LV4G: track 46.9 -> 0.00 mm, vias 2 -> 0
- net LV5G: track 45.8 -> 0.00 mm, vias 2 -> 0
- net LV6G: track 45.4 -> 0.00 mm, vias 2 -> 0
- net BATT+: track 56.5 -> 15.2 mm
- net IBLGHT: track 0.00 -> 37.8 mm, vias 0 -> 4
- net FANOUT: track 34.8 -> 0.00 mm
- net LV1G: track 31.0 -> 0.00 mm
- net N$31: track 51.0 -> 26.7 mm
- net HV3CTLG: track 24.3 -> 0.00 mm
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- added copper zone on layer 16, net BATT+
- added copper zone on layer 16, net BATT+IN
- added copper zone on layer 16, net BATT-
- added copper zone on layer 1, net HEATSINK
