File: board.sch (EAGLE design)
At the start: 0 parts

Commit message: Schematics v1
Parts:
- added C1: 470u, rcl:CPOL-EUE3.5-8
- added C2, C3, C5: 0.1u, rcl:C-EUC0805
- added C4: 100n, rcl:C-EUC0805
- added D1, D3, D4, D5, D6: STTH4R02UY, diode:DIODE-SMB
- added F1, F2, F3: 1.6A, fuse:SHK20L
- added F4, F5, F9: 30V/1.6A, SparkFun-Fuses:PPTC_PTH
- added F6, F7, F8: 30V/4A, SparkFun-Fuses:PPTC_PTH
- added IC1: REG1117, burr-brown:REG1117
- added J1: LHBEAMOUT, SparkFun-Connectors:CONN_03SCREW
- added J10: ATEMP, SparkFun-Connectors:CONN_023.5MM
- added J11: HORNOUT, SparkFun-Connectors:CONN_023.5MM
- added J12: 12V_SUPPLY, SparkFun-Connectors:CONN_023.5MM
- added J13: STOPOUT, SparkFun-Connectors:CONN_023.5MM
- added J14: TURNOUT, SparkFun-Connectors:CONN_03SCREW
- added J15: FANOUT, SparkFun-Connectors:CONN_023.5MM
- added J16: BLIGHTOUT, SparkFun-Connectors:CONN_023.5MM
- added J17: AUXOUT, SparkFun-Connectors:CONN_023.5MM
- added J18: AUX, SparkFun-Connectors:CONN_023.5MM
- added J19: CAN, SparkFun-Connectors:CONN_023.5MM
- added J2: BATT, SparkFun-Connectors:CONN_023.5MM
- added J3: BLIGHT, SparkFun-Connectors:CONN_023.5MM
- added J4: LHBEAM, SparkFun-Connectors:CONN_03SCREW
- added J5: LRTURN, SparkFun-Connectors:CONN_03SCREW
- added J6: WARNING, SparkFun-Connectors:CONN_023.5MM
- added J7: HORN, SparkFun-Connectors:CONN_023.5MM
- added J8: BREAK, SparkFun-Connectors:CONN_023.5MM
- added J9: ABREAK, SparkFun-Connectors:CONN_023.5MM
- added L1: 15uH, inductor-bourns:SDR1307
- added Q1, Q2, Q3: IRF7465TR, transistor-power:N-MOSFET-SO8S
- added Q4: IRLML9301TRPBF, svetozar:IRLML9301TRPBF
- added Q5, Q9: IRLML9301TRPBF, my:IRLML9301TRPBF
- added Q6, Q7, Q8: IRF7424TRPBF, transistor-power:P-MOSFET-SO8
- added R1, R2, R3: 160, rcl:R-EU_R0805
- added R10, R11, R12, R4, R5, R6, R7, R8, R9: 1k, rcl:R-EU_R0805
- added R13: 3k, rcl:R-EU_R0805
- added R14: 2.4k, rcl:R-EU_R0805
- added R15: 10k, rcl:R-EU_R0805
- added U$1: (no value), BluePill:BLUE_PILL
- added U1, U2, U3: VOM1271T, VOM1271T:VOM1271T
- added U4: MC14504BDR2G, MC14504BDR2G:MC14504BDR2G
- added U5: MAX3051ESA, MAX3051ESA:MAX3051ESA
Connections:
- new net +12V: C2.1, F4.2, F5.2, F6.2, F7.2, F8.2, F9.2, IC1.VIN, J12.1, U4.VDD
- new net +3V3: C3.1, C5.1, IC1.VOUT, R10.1, R11.1, R12.1, R14.1, R4.1, R5.1, R6.1, R7.1, R8.1, R9.1, U$1.3.3V, U$1.3.3V1, U4.VCC, U5.VCC
- new net AUXOUT: D1.C, J17.1, Q8.D
- new net BATT+: F1.2A, F2.2A, F3.2A, J2.1
- new net BATT-: D4.A, D5.A, D6.A, J1.3, J11.2, J2.2
- new net BLIGHTOUT: J16.1, Q7.D
- new net CANH: J19.1, U5.CANH
- new net CANL: J19.2, U5.CANL
- new net FANOUT: C1.+, D3.C, J15.1, L1.2
- new net GND: C4.2, C5.2, J10.1, J18.1, J3.1, J4.1, J5.1, J6.1, J7.1, J8.1, J9.1, R15.2, U5.GND, U5.RS
- new net GND1: C1.-, C2.2, C3.2, D1.A, D3.A, IC1.GND, J12.2, J13.2, J14.3, J15.2, J16.2, J17.2, U$1.GND, U$1.GND1, U$1.GND2, U1.C1, U2.C1, U3.C1, U4.MODE, U4.VSS
- new net HBEAMOUT: D5.C, J1.2, Q2.S, U2.C2
- new net HORNOUT: D6.C, J11.1, Q3.S, U3.C2
- new net HV1CTL: R1.1, U$1.PB1
- new net HV2CTL: R2.1, U$1.PB0
- new net HV3CTL: R3.1, U$1.PA7
- new net LBEAMOUT: D4.C, J1.1, Q1.S, U1.C2
- new net LTURNOUT: J14.1, Q5.D
- new net LVCTL1: U$1.PA6, U4.AIN
- new net N$1: U$1.PA3, U4.BIN
- new net N$10: F1.1A, Q1.D
- new net N$11: F2.1A, Q2.D
- new net N$12: F3.1A, Q3.D
- new net N$13: U$1.PB7, U4.EIN
- new net N$14: U$1.PB6, U4.FIN
- new net N$15: J3.2, R4.2, U$1.PA0
- new net N$16: F4.1, Q4.S
- new net N$17: L1.1, Q6.D
- new net N$18: F5.1, Q5.S
- new net N$19: F6.1, Q6.S
- new net N$2: U$1.PA2, U4.CIN
- new net N$20: Q4.G, U4.AOUT
- new net N$21: F7.1, Q7.S
- new net N$22: F8.1, Q8.S
- new net N$23: F9.1, Q9.S
- new net N$24: Q5.G, U4.BOUT
- new net N$25: Q9.G, U4.COUT
- new net N$26: Q6.G, U4.DOUT
- new net N$27: Q7.G, U4.EOUT
- new net N$28: Q8.G, U4.FOUT
- new net N$29: J4.3, R6.2, U$1.PB12
- new net N$3: U$1.PA1, U4.DIN
- new net N$30: J4.2, R5.2, U$1.PB13
- new net N$31: J7.2, R10.2, U$1.PA9
- new net N$32: J5.3, R8.2, U$1.PB14
- new net N$33: J5.2, R7.2, U$1.PB15
- new net N$34: J8.2, R11.2, U$1.PA10
- new net N$35: J6.2, R9.2, U$1.PA8
- new net N$36: J18.2, R12.2, U$1.PA15
- new net N$37: C4.1, J10.2, R14.2, U$1.PA4
- new net N$38: J9.2, R13.1
- new net N$39: R13.2, R15.1, U$1.PA5
- new net N$4: R1.2, U1.A1
- new net N$40: U$1.PB8, U5.RXD
- new net N$41: U$1.PB9, U5.TXD
- new net N$42: U$1.PB5, U5.SHDN
- new net N$5: R2.2, U2.A1
- new net N$6: R3.2, U3.A1
- new net N$7: Q1.G, U1.A2
- new net N$8: Q2.G, U2.A2
- new net N$9: Q3.G, U3.A2
- new net RTURNOUT: J14.2, Q9.D
- new net STOPOUT: J13.1, Q4.D

Commit message: PCB v.1
Parts:
- added C6: 470u, rcl:CPOL-EUE3.5-8
- added C7: 47u6V, rcl:C-EUC1206
- added C8: 22u16V, rcl:C-EUC1206
- added LOGO2: OSHW-LOGOL, SparkFun-Aesthetics:OSHW-LOGOL
- added R16: 120, rcl:R-EU_R0805
- C4: value 100n -> 0.1u
- F6, F7, F8: value 30V/4A -> 30V4A; device SparkFun-Fuses:PPTC_PTH -> svetozar:PPTC_WIDE
- IC1: value REG1117 -> LM1117; device burr-brown:REG1117 -> svetozar:LM1117
- U5: value MAX3051ESA -> MAX3051ESA+T; device MAX3051ESA:MAX3051ESA -> MAX3051ESA:MAX3051ESA+T
Connections:
- net N$10 renamed HV1
- net N$11 renamed HV2
- net N$12 renamed HV3
- net N$40 renamed CANRX
- net N$41 renamed CANTX
- net N$42 renamed CANSHDN
- removed net GND1: C1.-, C2.2, C3.2, D1.A, D3.A, IC1.GND, J12.2, J13.2, J14.3, J15.2, J16.2, J17.2, U$1.GND, U$1.GND1, U$1.GND2, U1.C1, U2.C1, U3.C1, U4.MODE, U4.VSS
- net +12V: now also C6.+, C8.1
- net +3V3: now also C7.1, IC1.P$1
- net CANH: now also J19.2, R16.2; no longer J19.1
- net CANL: now also J19.1, R16.1; no longer J19.2
- net GND: now also C1.-, C2.2, C3.2, C6.-, C7.2, C8.2, D1.A, D3.A, IC1.GND, J12.2, J13.2, J14.3, J15.2, J16.2, J17.2, U$1.GND, U$1.GND1, U$1.GND2, U1.C1, U2.C1, U3.C1, U4.MODE, U4.VSS
- net N$1: now also U4.DIN; no longer U4.BIN
- net N$13: now also U4.BIN; no longer U4.EIN
- net N$14: now also U4.CIN; no longer U4.FIN
- net N$2: now also U4.EIN; no longer U4.CIN
- net N$24: now also Q9.G; no longer Q5.G
- net N$25: now also Q5.G; no longer Q9.G
- net N$26: now also U4.EOUT; no longer U4.DOUT
- net N$27: now also U4.DOUT; no longer U4.EOUT
- net N$29: now also U$1.PB13; no longer U$1.PB12
- net N$3: now also U4.FIN; no longer U4.DIN
- net N$30: now also U$1.PB12; no longer U$1.PB13
- net N$32: now also U$1.PB15; no longer U$1.PB14
- net N$33: now also U$1.PB14; no longer U$1.PB15

Commit message: Board & schematics v 1.1. Minor improvements
Parts:
- C2: device rcl:C-EUC0805 -> rcl:C-EUC1206
Connections:
- net N$1 renamed LVCTL4
- net N$13 renamed LVCTL2
- net N$14 renamed LVCTL3
- net N$2 renamed LVCTL5
- net N$20 renamed LV4G
- net N$24 renamed LV5G
- net N$25 renamed LV6G
- net N$26 renamed LV3G
- net N$27 renamed LV2G
- net N$28 renamed LV1G
- net N$3 renamed LVCTL6
- net N$37 renamed IATEMP
- net N$38 renamed ABRK
- net N$39 renamed ABRK_S
- net N$4 renamed HV1CTLG
- net N$5 renamed HV2CTLG
- net N$6 renamed HV3CTLG
- net N$7 renamed HV1G
- net N$8 renamed HV2G
- net N$9 renamed HV3G
- net HV1CTL: now also U$1.PB0; no longer U$1.PB1
- net HV2CTL: now also U$1.PB1; no longer U$1.PB0
Changed lines of the file:
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@@
 </spice>
 </part>
-<part name="C2" library="rcl" library_urn="urn:adsk.eagle:library:334" deviceset="C-EU" device="C0805" package3d_urn="urn:adsk.eagle:package:23617/2" value="0.1u"/>
+<part name="C2" library="rcl" library_urn="urn:adsk.eagle:library:334" deviceset="C-EU" device="C1206" package3d_urn="urn:adsk.eagle:package:23618/2" value="0.1u"/>
 <part name="C3" library="rcl" library_urn="urn:adsk.eagle:library:334" deviceset="C-EU" device="C0805" package3d_urn="urn:adsk.eagle:package:23617/2" value="0.1u"/>
 <part name="LOGO2" library="SparkFun-Aesthetics" deviceset="OSHW-LOGO" device="L"/>
@@
 <net name="HV1CTL" class="0">
 <segment>
+<pinref part="R1" gate="G$1" pin="1"/>
+<wire x1="-20.32" y1="114.3" x2="-20.32" y2="157.48" width="0.1524" layer="91"/>
+<pinref part="U$1" gate="G$1" pin="PB0"/>
+<wire x1="-20.32" y1="114.3" x2="-60.96" y2="114.3" width="0.1524" layer="91"/>
+</segment>
+</net>
+<net name="HV2CTL" class="0">
+<segment>
+<pinref part="R2" gate="G$1" pin="1"/>
 <pinref part="U$1" gate="G$1" pin="PB1"/>
-<wire x1="-60.96" y1="116.84" x2="-20.32" y2="116.84" width="0.1524" layer="91"/>
-<pinref part="R1" gate="G$1" pin="1"/>
-<wire x1="-20.32" y1="116.84" x2="-20.32" y2="157.48" width="0.1524" layer="91"/>
-</segment>
-</net>
-<net name="HV2CTL" class="0">
-<segment>
-<pinref part="U$1" gate="G$1" pin="PB0"/>
-<wire x1="-60.96" y1="114.3" x2="-17.78" y2="114.3" width="0.1524" layer="91"/>
-<wire x1="-17.78" y1="114.3" x2="-17.78" y2="119.38" width="0.1524" layer="91"/>
-<pinref part="R2" gate="G$1" pin="1"/>
+<wire x1="-17.78" y1="116.84" x2="-17.78" y2="119.38" width="0.1524" layer="91"/>
+<wire x1="-60.96" y1="116.84" x2="-17.78" y2="116.84" width="0.1524" layer="91"/>
 </segment>
 </net>
@@
 </segment>
 </net>
-<net name="N$5" class="0">
+<net name="HV2CTLG" class="0">
 <segment>
 <pinref part="U2" gate="G$1" pin="A1"/>
@@
 </segment>
 </net>
-<net name="N$6" class="0">
+<net name="HV3CTLG" class="0">
 <segment>
 <pinref part="U3" gate="G$1" pin="A1"/>
@@
 </segment>
 </net>
-<net name="N$4" class="0">
+<net name="HV1CTLG" class="0">
 <segment>
 <pinref part="R1" gate="G$1" pin="2"/>
@@
 </segment>
 </net>
-<net name="N$7" class="0">
+<net name="HV1G" class="0">
 <segment>
 <pinref part="U1" gate="G$1" pin="A2"/>
@@
 </segment>
 </net>
-<net name="N$8" class="0">
+<net name="HV2G" class="0">
 <segment>
 <pinref part="U2" gate="G$1" pin="A2"/>
@@
 </segment>
 </net>
-<net name="N$9" class="0">
+<net name="HV3G" class="0">
 <segment>
 <pinref part="U3" gate="G$1" pin="A2"/>
@@
 </segment>
 </net>
-<net name="N$1" class="0">
+<net name="LVCTL4" class="0">
 <segment>
 <pinref part="U$1" gate="G$1" pin="PA3"/>
@@
 </segment>
 </net>
-<net name="N$2" class="0">
+<net name="LVCTL5" class="0">
 <segment>
 <pinref part="U$1" gate="G$1" pin="PA2"/>
@@
 </segment>
 </net>
-<net name="N$3" class="0">
+<net name="LVCTL6" class="0">
 <segment>
 <pinref part="U$1" gate="G$1" pin="PA1"/>
@@
 </segment>
 </net>
-<net name="N$13" class="0">
+<net name="LVCTL2" class="0">
 <segment>
 <pinref part="U$1" gate="G$1" pin="PB7"/>
@@
 </segment>
 </net>
-<net name="N$14" class="0">
+<net name="LVCTL3" class="0">
 <segment>
 <pinref part="U$1" gate="G$1" pin="PB6"/>
@@
 </segment>
 </net>
-<net name="N$20" class="0">
+<net name="LV4G" class="0">
 <segment>
 <pinref part="U4" gate="A" pin="AOUT"/>
@@
 </segment>
 </net>
-<net name="N$24" class="0">
+<net name="LV5G" class="0">
 <segment>
 <pinref part="U4" gate="A" pin="BOUT"/>
@@
 </segment>
 </net>
-<net name="N$25" class="0">
+<net name="LV6G" class="0">
 <segment>
 <pinref part="U4" gate="A" pin="COUT"/>
@@
 </segment>
 </net>
-<net name="N$26" class="0">
+<net name="LV3G" class="0">
 <segment>
 <pinref part="Q6" gate="G$1" pin="G"/>
@@
 </segment>
 </net>
-<net name="N$27" class="0">
+<net name="LV2G" class="0">
 <segment>
 <wire x1="-27.94" y1="48.26" x2="-27.94" y2="-35.56" width="0.1524" layer="91"/>
@@
 </segment>
 </net>
-<net name="N$28" class="0">
+<net name="LV1G" class="0">
 <segment>
 <pinref part="U4" gate="A" pin="FOUT"/>
@@
 </segment>
 </net>
-<net name="N$37" class="0">
+<net name="IATEMP" class="0">
 <segment>
 <pinref part="J10" gate="G$1" pin="2"/>
@@
 </segment>
 </net>
-<net name="N$38" class="0">
+<net name="ABRK" class="0">
 <segment>
 <pinref part="J9" gate="G$1" pin="2"/>
@@
 </segment>
 </net>
-<net name="N$39" class="0">
+<net name="ABRK_S" class="0">
 <segment>
 <pinref part="R13" gate="G$1" pin="2"/>

Commit message: Added BOM
Parts:
- C1, C6: MPN (none) -> SK016M0470B3F-0811; PRICE (none) -> 2,70р; SHOP (none) -> https://www.terraelectronica.ru/product/1262453
- C2: MPN (none) -> CC1206KRX7R8BB104; PRICE (none) -> 2,20р; SHOP (none) -> https://www.terraelectronica.ru/product/540763
- C3: MPN (none) -> CC0805KRX7R9BB104; PRICE (none) -> 2,00р; SHOP (none) -> https://www.terraelectronica.ru/product/251110
- C7: MPN CL31A476MQHNNNE -> CL31A476MQHNNNE; PRICE (none) -> 7,70р; SHOP (none) -> https://www.terraelectronica.ru/product/882710
- C8: MPN CL32A226KOJNNNE -> CL31A226KOHNNNE; PRICE (none) -> 12,80р; SHOP (none) -> https://www.terraelectronica.ru/product/1641407
- D1, D3, D4, D5, D6: MPN STTH4R02UY -> STTH4R02U; PRICE (none) -> 14,10р; SHOP (none) -> https://www.terraelectronica.ru/product/450947
- F1, F2, F3: MPN (none) -> FC-001S; PRICE (none) -> 2,10р; QTY (none) -> 2; SHOP (none) -> https://www.terraelectronica.ru/product/2076693
- F4, F5, F9: PRICE (none) -> 5,40р; SHOP (none) -> https://www.terraelectronica.ru/product/1040513
- F6, F7, F8: PRICE (none) -> 25,90р; SHOP (none) -> https://www.terraelectronica.ru/product/577123
- IC1: MPN (none) -> LD1117S33TR; PRICE (none) -> 12,00р; SHOP (none) -> https://www.terraelectronica.ru/product/208059
- J1, J14, J4, J5: MPN (none) -> DG350-3.5-03P-14-00AH; PRICE (none) -> 9,40р; SHOP (none) -> https://www.terraelectronica.ru/product/1108750
- J10, J11, J12, J13, J15, J16, J17, J18, J19, J2, J3, J6, J7, J8, J9: MPN (none) -> DG350-3.5-02P-14-00AH; PRICE (none) -> 5,80р; SHOP (none) -> https://www.terraelectronica.ru/product/1115132
- L1: MPN (none) -> SDR1307-150ML; PRICE (none) -> 21,20р; SHOP (none) -> https://www.terraelectronica.ru/product/607745
- Q1, Q2, Q3: MPN (none) -> IRF7465TRPBF; PRICE (none) -> 26,30р; SHOP (none) -> https://www.terraelectronica.ru/product/507651
- Q4, Q5, Q9: MPN (none) -> IRLML9301TRPBF; PRICE (none) -> 9,10р; SHOP (none) -> https://www.terraelectronica.ru/product/575910
- Q6, Q7, Q8: MPN (none) -> IRF7424TRPBF; PRICE (none) -> 15,40р; SHOP (none) -> https://www.terraelectronica.ru/product/301875
- R1: PRICE (none) -> 0,52р; SHOP (none) -> https://www.terraelectronica.ru/product/880371
- R13: MPN (none) -> RC0805JR-071KL; PRICE (none) -> 0,17р; SHOP (none) -> https://www.terraelectronica.ru/product/443003
- R14: MPN (none) -> RC0805FR-072K4L; PRICE (none) -> 0,15р; SHOP (none) -> https://www.terraelectronica.ru/product/562267
- R15: MPN (none) -> RC0805JR-0710KL; PRICE (none) -> 0,24р; SHOP (none) -> https://www.terraelectronica.ru/product/339147
- R16: MPN (none) -> RC0805FR-07120RL; PRICE (none) -> 0,23р; SHOP (none) -> https://www.terraelectronica.ru/product/542987
- R4: MPN (none) -> RC0805JR-071KL; PRICE (none) -> 0,19р; SHOP (none) -> https://www.terraelectronica.ru/product/559515
- U$1: MPN (none) -> Blue Pill; PRICE (none) -> 127,73р; SHOP (none) -> https://ru.aliexpress.com/item/STM32F103C8T6-ARM-STM32-Mini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
- U1, U2, U3: MPN (none) -> VOM1271T; PRICE (none) -> 173,00р; SHOP (none) -> https://www.terraelectronica.ru/product/1112827
- U4: MPN (none) -> MC14504BDR2G; PRICE (none) -> 25,70р; SHOP (none) -> https://www.terraelectronica.ru/product/284776
- U5: MPN (none) -> MAX3051ESA+T; PRICE (none) -> 141,00р; SHOP (none) -> https://www.terraelectronica.ru/product/462120

Commit message: WIP
Parts:
- removed F1, F2, F3: 1.6A, fuse:SHK20L
- removed F4, F5, F9: 30V/1.6A, SparkFun-Fuses:PPTC_PTH
- removed F6, F7, F8: 30V4A, svetozar:PPTC_WIDE
- added C10, C9: 1n, rcl:C-EUC0805
- added C11, C12: 0.1u, rcl:C-EUC0805
- added JP1: (no value), jumper:JP1E
- added JP2: (no value), jumper:JP2E
- added LED1: (no value), led:LEDSML0805
- added R17: 1k, rcl:R-EU_R0603
- added R18, R19, R20, R21, R22, R23: 10k, rcl:R-EU_R0603
- added U$2, U$3: ACS711LC, svetozar:ACS711
- C1, C6: device rcl:CPOL-EUE3.5-8 -> rcl:CPOL-EUF
- IC1: value LM1117 -> REG1117F; device svetozar:LM1117 -> burr-brown:REG1117F
- J10: value ATEMP -> TEMP
- J8: value BREAK -> (none); device SparkFun-Connectors:CONN_023.5MM -> SparkFun-Connectors:CONN_01; MPN DG350-3.5-02P-14-00AH -> (none); PRICE 5,80р -> (none); SHOP https://www.terraelectronica.ru/product/1115132 -> (none)
- J9: value ABREAK -> BREAK; device SparkFun-Connectors:CONN_023.5MM -> SparkFun-Connectors:CONN_03SCREW
- Q1, Q2, Q3: value IRF7465TR -> FQD19N10LTM; device transistor-power:N-MOSFET-SO8S -> SparkFun-DiscreteSemi:MOSFET-NCH-FDD8780; MPN IRF7465TRPBF -> FQD19N10LTM; PRICE 26,30р -> 15,80р; SHOP https://www.terraelectronica.ru/product/507651 -> https://www.terraelectronica.ru/product/675613
- Q4: value IRLML9301TRPBF -> IRF7424TRPBF; device svetozar:IRLML9301TRPBF -> transistor-power:P-MOSFET-SO8
- Q5, Q9: value IRLML9301TRPBF -> IRF7424TRPBF; device my:IRLML9301TRPBF -> transistor-power:P-MOSFET-SO8
- R10, R12, R13, R14, R15, R4, R5, R6, R7, R8, R9: device rcl:R-EU_R0805 -> rcl:R-EU_R0603
Connections:
- net ABRK renamed N$5
- removed net CANL: J19.1, R16.1, U5.CANL
- removed net HV1: F1.1A, Q1.D
- removed net HV2: F2.1A, Q2.D
- removed net HV3: F3.1A, Q3.D
- removed net N$15: J3.2, R4.2, U$1.PA0
- removed net N$16: F4.1, Q4.S
- removed net N$18: F5.1, Q5.S
- removed net N$19: F6.1, Q6.S
- removed net N$21: F7.1, Q7.S
- removed net N$22: F8.1, Q8.S
- removed net N$23: F9.1, Q9.S
- removed net N$34: J8.2, R11.2, U$1.PA10
- removed net N$36: J18.2, R12.2, U$1.PA15
- new net BATT+IN: J2.1, U$2.IP+@1, U$2.IP+@2
- new net CSENS1: C9.1, U$1.PA0, U$2.VOUT
- new net FAULT: R11.1, U$1.PB3, U$2.!FAULT, U$3.!FAULT
- new net IAUX: J18.2, R12.2, U$1.PB4
- new net IBLGHT: J3.2, R4.2, U$1.PB11
- new net N$1: JP1.2, R16.1
- new net N$2: J19.1, JP1.1, U5.CANL
- new net N$3: JP2.1, R13.2, R15.1
- new net N$4: J9.3, JP2.3, R17.2
- new net N$6: J8.1, LED1.A, U$1.PB10
- new net N$7: J12.1, U$3.IP+@1, U$3.IP+@2
- new net N$8: C10.1, U$1.PA6, U$3.VOUT
- new net N$9: C11.1, C12.1, U$1.PA15, U$2.VCC, U$3.VCC
- net +12V: now also Q4.S, Q5.S, Q6.S, Q7.S, Q8.S, Q9.S, U$3.IP-@3, U$3.IP-@4; no longer F4.2, F5.2, F6.2, F7.2, F8.2, F9.2, J12.1
- net +3V3: now also R11.2, R17.1, R18.2, R19.2, R20.2, R21.2, R22.2, R23.2; no longer IC1.P$1, R11.1
- net ABRK_S: now also JP2.2; no longer R13.2, R15.1
- net BATT+: now also Q1.D, Q2.D, Q3.D, U$2.IP-@3, U$2.IP-@4; no longer F1.2A, F2.2A, F3.2A, J2.1
- net FANOUT: no longer D3.C
- net GND: now also C10.2, C11.2, C12.2, C9.2, LED1.C, U$2.GND, U$3.GND; no longer J8.1
- net LVCTL1: now also R23.1, U$1.PA10; no longer U$1.PA6
- net LVCTL2: now also R22.1
- net LVCTL3: now also R21.1
- net LVCTL4: now also R20.1
- net LVCTL5: now also R19.1
- net LVCTL6: now also R18.1
- net N$17: now also D3.C
Other:
- moved on the sheet: C2, C3, C4, C5, C6, C7, C8, D3, J10, J12, J13, J14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
