File: board.sch (EAGLE design)
At the start: 81 parts, among them IC1 LD1117V33, J1 BLIGHT, J10 BATT, J11 LHBEAMOUT, J12 HORHOUT, J13 12V_SUPPLY, J14 STOPOUT, J15 TURNOUT, J16 FANOUT, J17 BLIGHTOUT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

Commit message: minor v2 fixes
Parts:
- R20, R21, R22: MPN RC0805FR-07160RL -> RC0603FR-07160RL
Changed lines of the file:
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@@
 </part>
 <part name="R20" library="SparkFun-Resistors" deviceset="RESISTOR" device="0603" value="160">
-<attribute name="MPN" value="RC0805FR-07160RL"/>
+<attribute name="MPN" value="RC0603FR-07160RL"/>
 </part>
 <part name="R21" library="SparkFun-Resistors" deviceset="RESISTOR" device="0603" value="160">
-<attribute name="MPN" value="RC0805FR-07160RL"/>
+<attribute name="MPN" value="RC0603FR-07160RL"/>
 </part>
 <part name="R22" library="SparkFun-Resistors" deviceset="RESISTOR" device="0603" value="160">
-<attribute name="MPN" value="RC0805FR-07160RL"/>
+<attribute name="MPN" value="RC0603FR-07160RL"/>
 </part>
 <part name="SUPPLY4" library="supply2" library_urn="urn:adsk.eagle:library:372" deviceset="GND" device=""/>
